File: Hardware/Base_Step_down/Helena_base_sd.kicad_pcb (KiCad board)
At the start: 2 copper layers, 38 x 18 mm, 56 parts, among them IC1 ATTINY85-S, P1 CONN_01X01, P2 CONN_01X01, P3 CONN_01X01, P4 CONN_01X06, P5 CONN_01X01, P6 CONN_01X01, P7 CONN_01X01, P8 CONN_01X01, Q1 BC857C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

Commit message: added reverse polarity protection and led board
Parts:
- added Q6: IRLML0030, footprints:SOT-23, B.Cu at (62.9, 144.0)
- added Q7: IRLML0030, footprints:SOT-23, B.Cu at (62.9, 147.3)
- added R14: 10k, rt_device:C_0603_THERMaL_RELIEF, B.Cu at (65.4, 145.7)
- C13, C2: value 150n -> 100n
- Q3, Q4: value IRLML6246 -> IRLML0030
Connections:
- P3 pad 1: GND -> Net-(P3-Pad1)
Routing:
- net VPP: track 102.4 -> 92.9 mm
- net GND: track 81.7 -> 74.1 mm, vias 28 -> 24
- net Net-(P3-Pad1): track 0.00 -> 6.29 mm, vias 0 -> 4
- net Net-(Q6-Pad1): track 0.00 -> 5.85 mm
- added copper zone on F.Cu, net Net-(P2-Pad1)
- added copper zone on B.Cu, net Net-(P3-Pad1)
- added copper zone on F.Cu, net Net-(P3-Pad1)
- added copper zone on B.Cu, net VPP
Other:
- board text added: "RT1702"
- board text removed: "RT1612"
