File: Hardware/Base_Step_down/Helena_base_sd.sch (KiCad schematic (older format))
At the start: 53 parts, among them IC1 ATTINY85-S, P1 CONN_01X01, P2 CONN_01X01, P3 CONN_01X01, P4 CONN_01X06, P5 CONN_01X01, P6 CONN_01X01, P7 CONN_01X01, P8 CONN_01X01, Q1 BC857C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

Commit message: added reverse polarity protection and led board
Parts:
- added Q6, Q7: IRLML0030, footprints:SOT-23, symbol Q_NMOS_GSD
- added R14: 10k, rt_device:C_0603_THERMaL_RELIEF, symbol R
- C13, C2: value 150n -> 100n
- IC1: symbol ATTINY85-S -> ATTINY85-S-RESCUE-Helena_base_sd
- Q3, Q4: value IRLML6246 -> IRLML0030
Connections:
- net GND: now also Q6.2 (S), Q7.2 (S); no longer P3.1 (P1)
- net VPP: now also R14.2
- new net: P3.1 (P1), Q6.3 (D), Q7.3 (D)
- new net: Q6.1 (G), Q7.1 (G), R14.1
Other:
- note removed: "2.2"
- note removed: "2016/12/15"
- note removed: "Dual 3.0A Step Down LED Driver"
- note removed: "Helena Base Step Down"
- note removed: "Helena base"
- moved on the sheet: C10, C12, C4, D2, FB1, IC1, P1, P2, P3, Q2, R2, R3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

Commit message: Hardware update for better compatibility with KD2 style lights
Parts:
- C1, C10, C11, C12, C13, C14, C2, C3, C4, C7: footprint rt_device:C_0603_THERMaL_RELIEF -> Capacitor_SMD:C_0603_1608Metric; symbol C -> Helena_base_sd-rescue:C
- C5, C9: footprint Capacitors_SMD:C_0805 -> Capacitor_SMD:C_0805_2012Metric; symbol C -> Helena_base_sd-rescue:C
- C6, C8: footprint Capacitors_SMD:C_1206 -> Capacitor_SMD:C_1206_3216Metric; symbol C -> Helena_base_sd-rescue:C
- D1, D2, D4, D7: footprint TO_SOT_Packages_SMD:SOT-23 -> Package_TO_SOT_SMD:SOT-23; symbol ZENER_3pin_KNCA -> Helena_base_sd-rescue:ZENER_3pin_KNCA
- D3, D6: footprint rt_diodes:SMA -> rt_diodes:D_SMA; symbol D_Schottky -> Helena_base_sd-rescue:D_Schottky
- D5: footprint TO_SOT_Packages_SMD:SOT-23 -> Package_TO_SOT_SMD:SOT-23; symbol D_Schottky_x2_ACom_KKA -> Helena_base_sd-rescue:D_Schottky_x2_ACom_KKA
- FB1: footprint rt_device:C_0603_THERMaL_RELIEF -> Inductor_SMD:L_0603_1608Metric; symbol FB -> Helena_base_sd-rescue:FB
- L1, L2: symbol INDUCTOR_SMALL -> Helena_base_sd-rescue:INDUCTOR_SMALL
- P1, P2, P3, P5, P6, P7, P8: symbol CONN_01X01 -> Helena_base_sd-rescue:CONN_01X01
- P4: symbol CONN_01X06 -> Helena_base_sd-rescue:CONN_01X06
- Q1, Q5: footprint TO_SOT_Packages_SMD:SOT-23 -> Package_TO_SOT_SMD:SOT-23; symbol Q_PNP_BEC -> Helena_base_sd-rescue:Q_PNP_BEC
- Q2, Q3, Q4: footprint TO_SOT_Packages_SMD:SOT-23 -> Package_TO_SOT_SMD:SOT-23; symbol Q_NMOS_GSD -> Helena_base_sd-rescue:Q_NMOS_GSD
- Q6, Q7: footprint footprints:SOT-23 -> Package_TO_SOT_SMD:SOT-23; symbol Q_NMOS_GSD -> Helena_base_sd-rescue:Q_NMOS_GSD
- R1, R10, R11, R12, R13, R14, R2, R3, R4, R5, R6, R7, R8, R9: footprint rt_device:C_0603_THERMaL_RELIEF -> Resistor_SMD:R_0603_1608Metric; symbol R -> Helena_base_sd-rescue:R
- U1: footprint Housings_SSOP:MSOP-8_3x3mm_Pitch0.65mm -> Package_SO:MSOP-8_3x3mm_P0.65mm; symbol MCP6482 -> Helena_base_sd-rescue:MCP6482
- U2: footprint TO_SOT_Packages_SMD:SOT-23 -> Package_TO_SOT_SMD:SOT-23W; symbol MCP1703 -> Helena_base_sd-rescue:MCP1703
- U3: renamed from IC1; footprint rt_Housings_SOIC:SOIC-8_5.29x4.9mm_Pitch1.27mm -> Package_SO:SOIC-8_5.23x5.23mm_P1.27mm; symbol ATTINY85-S-RESCUE-Helena_base_sd -> Helena_base_sd-rescue:ATTINY85-S-RESCUE-Helena_base_sd
