File: Hardware/Ctrl/Helena_ctrl.sch (KiCad schematic (older format))
At the start: 36 parts, among them P1 CONN_01X06, P2 CONN_01X04, Q1 BC857C, SW1 SW_PUSH, U1 antenna-gnd, U2 nrf51822-qfax, U3 MPU-6050, Y1 16MHz

Commit message: added reverse polarity protection and led board
Parts:
- C11: value 47n -> 100n
- R3, R5: value 3k3 -> 1k5
- R4: value 560 -> 680
Other:
- note removed: "2.1"
- note removed: "2016/12/15"
- note removed: "Bluetooth Control Board"
- note removed: "Helena"
- note removed: "Helena Ctrl"
Changed lines of the file:
@@
 LIBS:contrib
 LIBS:valves
-LIBS:rt_logos
 LIBS:Helena_ctrl-cache
 EELAYER 25 0
@@
 encoding utf-8
 Sheet 1 1
-Title ""
-Date ""
-Rev ""
+Title "Helena Wireless Control Board"
+Date "2016-12-15"
+Rev "2.1"
 Comp ""
 Comment1 ""
@@
 P 3000 5250
 F 0 "C11" H 3025 5350 50  0000 L CNN
-F 1 "47n" H 3025 5150 50  0000 L CNN
+F 1 "100n" H 3025 5150 50  0000 L CNN
 F 2 "rt_device:C_0603_THERMaL_RELIEF" H 3038 5100 30  0001 C CNN
 F 3 "" H 3000 5250 60  0000 C CNN
@@
 P 9200 1850
 F 0 "R3" V 9280 1850 50  0000 C CNN
-F 1 "3k3" V 9200 1850 50  0000 C CNN
+F 1 "1k5" V 9200 1850 50  0000 C CNN
 F 2 "rt_device:C_0603_THERMaL_RELIEF" V 9130 1850 30  0001 C CNN
 F 3 "" H 9200 1850 30  0000 C CNN
@@
 P 9400 1850
 F 0 "R5" V 9480 1850 50  0000 C CNN
-F 1 "3k3" V 9400 1850 50  0000 C CNN
+F 1 "1k5" V 9400 1850 50  0000 C CNN
 F 2 "rt_device:C_0603_THERMaL_RELIEF" V 9330 1850 30  0001 C CNN
 F 3 "" H 9400 1850 30  0000 C CNN
@@
 P 9100 5350
 F 0 "R4" V 9180 5350 50  0000 C CNN
-F 1 "560" V 9100 5350 50  0000 C CNN
+F 1 "680" V 9100 5350 50  0000 C CNN
 F 2 "rt_device:C_0603_THERMaL_RELIEF" V 9030 5350 30  0001 C CNN
 F 3 "" H 9100 5350 30  0000 C CNN
@@
 NoConn ~ 5100 5100
 NoConn ~ 5100 5200
-$Comp
-L Helena #G?
-U 1 1 5852E504
-P 7300 6850
-F 0 "#G?" H 7300 6631 60  0001 C CNN
-F 1 "Helena" H 7300 7069 60  0001 C CNN
-F 2 "" H 7300 6850 60  0000 C CNN
-F 3 "" H 7300 6850 60  0000 C CNN
-	1    7300 6850
-	1    0    0    -1
-$EndComp
-Text Notes 7650 6950 0    250  ~ 0
-Helena
-Text Notes 7700 7050 0    60   ~ 0
-Bluetooth Control Board
-Text Notes 7400 7500 0    60   ~ 0
-Helena Ctrl
-Text Notes 8140 7640 0    60   ~ 0
-2016/12/15
-Text Notes 10570 7645 0    60   ~ 0
-2.1
 $EndSCHEMATC

Commit message: updated control board
Parts:
- removed C10, C7: 22p, rt_device:C_0603_THERMaL_RELIEF, symbol C
- removed C11, C12, C3, C4: 100n, rt_device:C_0603_THERMaL_RELIEF, symbol C
- removed C5: 1p0, rt_device:C_0603_THERMaL_RELIEF, symbol C
- removed C6: 1n, rt_device:C_0603_THERMaL_RELIEF, symbol C
- removed C8: 2p2, rt_device:C_0603_THERMaL_RELIEF, symbol C
- removed C9: 2n2, rt_device:C_0603_THERMaL_RELIEF, symbol C
- removed D1: Double_LED, rt_leds:Duo-Led_0603, symbol Double_LED
- removed L1: 3n3, rt_device:C_0603_THERMaL_RELIEF, symbol INDUCTOR_SMALL
- removed L2: 4n7, rt_device:C_0603_THERMaL_RELIEF, symbol INDUCTOR_SMALL
- removed L3: 10n, rt_device:C_0603_THERMaL_RELIEF, symbol INDUCTOR_SMALL
- removed P2: CONN_01X04, rt_Pin_Header:Pin_Header_Straight_1x04_Pitch1.27mm, symbol CONN_01X04
- removed Q1: BC857C, TO_SOT_Packages_SMD:SOT-23, symbol Q_PNP_BEC
- removed U1: antenna-gnd, rt_antennas:MML_R302.302.000, symbol antenna-gnd
- removed U2: nrf51822-qfax, Housings_DFN_QFN:UQFN-48-1EP_6x6mm_Pitch0.4mm, symbol nrf51822-qfax
- removed Y1: 16MHz, rt_XTAL:XTAL_MT_3.2mm_x_2.5mm, symbol Crystal_4pin
- added D1: LED_RED, rt_device:C_0603_THERMaL_RELIEF, symbol LED
- added D2: LED_BLUE, rt_device:C_0603_THERMaL_RELIEF, symbol LED
- added FB2: FB, rt_device:C_0603_THERMaL_RELIEF, symbol FB
- added P2: CONN_02X05, rt_Pin_Header:Pin_Header_Straight_2x05_Pitch1.27mm, symbol CONN_02X05
- added U2: nrf51822-04AT_Module, rt_modules:WT51822-S4AT, symbol nrf51822-04AT_Module
- C1: value dnp -> 2u2/16
- C2: value 1p5 -> 100n
Connections:
- net LED_RED is gone; now on net +3V3: R4.1
- net +3V3: now also FB2.2, P2.1 (P1)
- net BDEP_RX: now also U2.8 (RESET/P0.10)
- net BUTTON: now also U2.7 (ENABLE/P0.09)
- net GND: now also R7.2, P2.3 (P3), P2.5 (P5), P2.9 (P9), U2.12 (GND), U2.13 (GND), U2.15 (ANT_GND), U2.2 (GND)
- net MPU_INT: now also U2.6 (TEST/P0.04)
- net SCL: now also U2.5 (INT/P0.03)
- net SDA: now also U2.4 (TXD/P0.02)
- net SWDCLK: now also P2.4 (P4), U2.11 (SWDCLK)
- net SWDIO: now also P2.2 (P2), U2.10 (SWDIO)
- net VIN_ADC: now also U2.3 (RXD/P0.01)
- net at C1.1, C2.1: now also FB2.1, U2.1 (VCC)
- net at R4.2: now also D1.2 (A)
- net LED_BLUE: no longer names the net of R7.1
- net LED_BLUE: now also D2.1 (K)
- new net ~LED_RED~/LED_BLUE: D1.1 (K), D2.2 (A), U2.9 (NC/P0.13)
- no-connect marks 26 -> 3
Other:
- moved on the sheet: C13, C14, C15, C16, C17, FB1, P1, R1, R2, R3, R4, R5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

Commit message: Hardware update for better compatibility with KD2 style lights
Parts:
- A1: renamed from U2; symbol nrf51822-04AT_Module -> Helena_ctrl-rescue:nrf51822-04AT_Module
- C1, C13, C14, C15, C16, C17, C2: footprint rt_device:C_0603_THERMaL_RELIEF -> Capacitor_SMD:C_0603_1608Metric; symbol C -> Helena_ctrl-rescue:C
- D1, D2: footprint rt_device:C_0603_THERMaL_RELIEF -> Diode_SMD:D_0603_1608Metric; symbol LED -> Helena_ctrl-rescue:LED
- FB1, FB2: footprint rt_device:C_0603_THERMaL_RELIEF -> Inductor_SMD:L_0603_1608Metric; symbol FB -> Helena_ctrl-rescue:FB
- J1: renamed from P1; footprint rt_Pin_Header:Pin_Header_Straight_1x06_2.00_Pitch -> Connector_PinHeader_2.00mm:PinHeader_1x06_P2.00mm_Vertical; symbol CONN_01X06 -> Helena_ctrl-rescue:CONN_01X06
- J2: renamed from P2; footprint rt_Pin_Header:Pin_Header_Straight_2x05_Pitch1.27mm -> Connector_PinHeader_1.27mm:PinHeader_2x05_P1.27mm_Vertical; symbol CONN_02X05 -> Helena_ctrl-rescue:CONN_02X05
- R1, R2, R3, R4, R5, R7: footprint rt_device:C_0603_THERMaL_RELIEF -> Resistor_SMD:R_0603_1608Metric; symbol R -> Helena_ctrl-rescue:R
- SW1: symbol SW_PUSH -> Helena_ctrl-rescue:SW_PUSH
- U1: renamed from U3; symbol MPU-6050 -> Helena_ctrl-rescue:MPU-6050
